File: tarefa1/tarefa1.sch (KiCad schematic (older format))
At the start: 13 parts, among them U1 nRF52832-QFxx, x1 32MHz

Commit message: Adicionando pcb
Parts:
- C1, C2, C3, C4, C5, C6, C7, C8: footprint (none) -> Capacitor_SMD:C_0402_1005Metric
- L1, L2, L3: footprint (none) -> Inductor_SMD:L_0402_1005Metric
- x1: footprint (none) -> Crystal:Crystal_SMD_3215-2Pin_3.2x1.5mm
Changed lines of the file:
@@
 EESchema Schematic File Version 4
+LIBS:tarefa1-cache
 EELAYER 29 0
 EELAYER END
@@
 F 0 "L2" H 6250 1665 50  0000 C CNN
 F 1 "10microH" H 6250 1574 50  0000 C CNN
-F 2 "" H 6250 1450 50  0001 C CNN
+F 2 "Inductor_SMD:L_0402_1005Metric" H 6250 1450 50  0001 C CNN
 F 3 "~" H 6250 1450 50  0001 C CNN
 	1    6250 1450
@@
 F 0 "C4" H 5022 1246 50  0000 R CNN
 F 1 "100nF" H 5022 1155 50  0000 R CNN
-F 2 "" H 5200 1200 50  0001 C CNN
+F 2 "Capacitor_SMD:C_0402_1005Metric" H 5200 1200 50  0001 C CNN
 F 3 "~" H 5200 1200 50  0001 C CNN
 	1    5200 1200
@@
 F 0 "L3" H 6850 1665 50  0000 C CNN
 F 1 "10nH" H 6850 1574 50  0000 C CNN
-F 2 "" H 6850 1450 50  0001 C CNN
+F 2 "Inductor_SMD:L_0402_1005Metric" H 6850 1450 50  0001 C CNN
 F 3 "~" H 6850 1450 50  0001 C CNN
 	1    6850 1450
@@
 F 0 "C3" H 7072 2396 50  0000 R CNN
 F 1 "100nF" H 7072 2305 50  0000 R CNN
-F 2 "" H 7250 2350 50  0001 C CNN
+F 2 "Capacitor_SMD:C_0402_1005Metric" H 7250 2350 50  0001 C CNN
 F 3 "~" H 7250 2350 50  0001 C CNN
 	1    7250 2350
@@
 F 0 "C5" V 5765 900 50  0000 C CNN
 F 1 "100nF" V 5674 900 50  0000 C CNN
-F 2 "" H 5450 900 50  0001 C CNN
+F 2 "Capacitor_SMD:C_0402_1005Metric" H 5450 900 50  0001 C CNN
 F 3 "~" H 5450 900 50  0001 C CNN
 	1    5450 900
@@
 F 0 "L1" H 3900 2965 50  0000 C CNN
 F 1 "10microH" H 3900 2874 50  0000 C CNN
-F 2 "" H 3900 2750 50  0001 C CNN
+F 2 "Inductor_SMD:L_0402_1005Metric" H 3900 2750 50  0001 C CNN
 F 3 "~" H 3900 2750 50  0001 C CNN
 	1    3900 2750
@@
 F 0 "C8" H 3672 3696 50  0000 R CNN
 F 1 "100nF" H 3672 3605 50  0000 R CNN
-F 2 "" H 3850 3650 50  0001 C CNN
+F 2 "Capacitor_SMD:C_0402_1005Metric" H 3850 3650 50  0001 C CNN
 F 3 "~" H 3850 3650 50  0001 C CNN
 	1    3850 3650
@@
 F 0 "C7" V 4165 1500 50  0000 C CNN
 F 1 "100pF" V 4074 1500 50  0000 C CNN
-F 2 "" H 3850 1500 50  0001 C CNN
+F 2 "Capacitor_SMD:C_0402_1005Metric" H 3850 1500 50  0001 C CNN
 F 3 "~" H 3850 1500 50  0001 C CNN
 	1    3850 1500
@@
 F 0 "C6" V 4165 2000 50  0000 C CNN
 F 1 "N.C." V 4074 2000 50  0000 C CNN
-F 2 "" H 3850 2000 50  0001 C CNN
+F 2 "Capacitor_SMD:C_0402_1005Metric" H 3850 2000 50  0001 C CNN
 F 3 "~" H 3850 2000 50  0001 C CNN
 	1    3850 2000
@@
 F 0 "x1" H 3128 3096 50  0000 L CNN
 F 1 "32MHz" H 3128 3005 50  0000 L CNN
-F 2 "" H 2950 3050 50  0001 C CNN
+F 2 "Crystal:Crystal_SMD_3215-2Pin_3.2x1.5mm" H 2950 3050 50  0001 C CNN
 F 3 "" H 2950 3050 50  0001 C CNN
 	1    2950 3050
@@
 F 0 "C1" V 2465 2650 50  0000 C CNN
 F 1 "12pF" V 2374 2650 50  0000 C CNN
-F 2 "" H 2150 2650 50  0001 C CNN
+F 2 "Capacitor_SMD:C_0402_1005Metric" H 2150 2650 50  0001 C CNN
 F 3 "~" H 2150 2650 50  0001 C CNN
 	1    2150 2650
@@
 F 0 "C2" V 2465 3450 50  0000 C CNN
 F 1 "12pF" V 2374 3450 50  0000 C CNN
-F 2 "" H 2150 3450 50  0001 C CNN
+F 2 "Capacitor_SMD:C_0402_1005Metric" H 2150 3450 50  0001 C CNN
 F 3 "~" H 2150 3450 50  0001 C CNN
 	1    2150 3450
