File: Medidor/Medidor.sch (KiCad schematic (older format))
At the start: 47 parts, among them J1 TC2030-CTX-TAG_CONECT, SW1 Rotary_Encoder_Switch, SW2 SW_DPST_x2, U1 INA219-INA, U2 Serial, X1 32MHz

Commit message: Add files via upload
Parts:
- ANT1: value 2450AT43B100E -> 2450AT18D0100
- D1: footprint (none) -> LED_SMD:LED_0603_1608Metric
- J1: footprint (none) -> Connector:Tag-Connect_TC2030-IDC-NL_2x03_P1.27mm_Vertical
- SW1: footprint (none) -> Rotary_Encoder:RotaryEncoder_Alps_EC11E-Switch_Vertical_H20mm
- U1: footprint SOT23-8 -> Package_TO_SOT_SMD:SuperSOT-8
- U2: symbol medidor:Serial -> Medidor-rescue:Serial-medidor
- dc1: footprint (none) -> Package_TO_SOT_SMD:SuperSOT-8
Connections:
- net R_B: now reaches R14.2, SW1.S1
- net Rx renamed RX
- net Tx renamed TX
Changed lines of the file:
@@
 F 0 "D1" V 3839 1583 50  0000 R CNN
 F 1 "LED" V 3748 1583 50  0000 R CNN
-F 2 "" H 3800 1700 50  0001 C CNN
+F 2 "LED_SMD:LED_0603_1608Metric" H 3800 1700 50  0001 C CNN
 F 3 "~" H 3800 1700 50  0001 C CNN
 	1    3800 1700
@@
 P 10000 5400
 F 0 "ANT1" H 10080 5389 50  0000 L CNN
-F 1 "2450AT43B100E" H 10080 5298 50  0000 L CNN
+F 1 " 2450AT18D0100" H 10080 5298 50  0000 L CNN
 F 2 "" H 10000 5400 50  0001 C CNN
 F 3 "~" H 10000 5400 50  0001 C CNN
@@
 F 0 "SW1" V 2000 4870 50  0000 R CNN
 F 1 "Rotary_Encoder_Switch" V 1955 4870 50  0001 R CNN
-F 2 "" H 1850 5260 50  0001 C CNN
+F 2 "Rotary_Encoder:RotaryEncoder_Alps_EC11E-Switch_Vertical_H20mm" H 1850 5260 50  0001 C CNN
 F 3 "~" H 2000 5360 50  0001 C CNN
 	1    2000 5100
@@
 F 0 "J1" H 5600 7517 50  0000 C CNN
 F 1 "TC2030-CTX-TAG_CONECT" H 5600 7426 50  0000 C CNN
-F 2 "" H 5600 7150 50  0001 C CNN
+F 2 "Connector:Tag-Connect_TC2030-IDC-NL_2x03_P1.27mm_Vertical" H 5600 7150 50  0001 C CNN
 F 3 "" H 5600 7150 50  0001 L BNN
 F 4 "None" H 5600 7150 50  0001 L BNN "Campo4"
@@
 F 0 "dc1" H 2225 7533 50  0001 C CNN
 F 1 "DC-DC" H 2225 7533 50  0000 C CNN
-F 2 "" H 2200 7300 50  0001 C CNN
+F 2 "Package_TO_SOT_SMD:SuperSOT-8" H 2200 7300 50  0001 C CNN
 F 3 "" H 2200 7300 50  0001 C CNN
 	1    2200 7300
@@
 F 0 "U1" H 9200 2717 50  0000 C CNN
 F 1 "INA219-INA" H 9200 2626 50  0000 C CNN
-F 2 "SOT23-8" H 9200 1850 50  0001 L BNN
+F 2 "Package_TO_SOT_SMD:SuperSOT-8" H 9200 1850 50  0001 L BNN
 F 3 "" H 9200 1850 50  0001 L BNN
 F 4 "SOT-23-8 Texas Instruments" H 9200 1850 50  0001 L BNN "Campo4"
@@
 	1550 4650 1550 4500
 $Comp
-L medidor:Serial U2
-U 1 1 5D3818B1
-P 4300 7050
-F 0 "U2" V 4196 7278 50  0000 L CNN
-F 1 "Serial" V 4287 7278 50  0000 L CNN
-F 2 "" H 4300 7050 50  0001 C CNN
-F 3 "" H 4300 7050 50  0001 C CNN
-	1    4300 7050
-	0    1    1    0
-$EndComp
-$Comp
 L power:Earth #PWR01
 U 1 1 5D384AF3
@@
 	3950 6800 3950 7000
 NoConn ~ 5200 5350
-Text GLabel 5300 5550 0    50   Input ~ 0
-Tx
 Wire Wire Line
 	5300 5550 5300 5350
-Text GLabel 5300 5650 0    50   Input ~ 0
-Rx
-Wire Wire Line
-	5300 5650 5400 5650
-Wire Wire Line
-	5400 5650 5400 5350
-Text GLabel 4200 6600 0    50   Input ~ 0
-Tx
-Wire Wire Line
-	4300 6800 4300 6600
 Wire Wire Line
 	4300 6600 4200 6600
-Text GLabel 4500 6600 2    50   Input ~ 0
-Rx
 Wire Wire Line
 	4500 6600 4400 6600
@@
 NoConn ~ 6100 3550
 NoConn ~ 6000 3550
+Wire Wire Line
+	1900 4650 1900 4450
+Wire Wire Line
+	1900 4450 2200 4450
+Connection ~ 1900 4650
+Text Label 2200 4450 0    50   ~ 0
+R_B
+$Comp
+L Medidor-rescue:Serial-medidor U2
+U 1 1 5D3818B1
+P 4300 7050
+F 0 "U2" V 4196 7278 50  0000 L CNN
+F 1 "Serial" V 4287 7278 50  0000 L CNN
+F 2 "" H 4300 7050 50  0001 C CNN
+F 3 "" H 4300 7050 50  0001 C CNN
+	1    4300 7050
+	0    1    1    0
+$EndComp
+Wire Wire Line
+	4300 6600 4300 6800
+Text Label 4200 6600 0    50   ~ 0
+TX
+Text Label 4500 6600 0    50   ~ 0
+RX
+Text Label 5300 5550 0    50   ~ 0
+TX
+Wire Wire Line
+	5400 5350 5400 5550
+Text Label 5400 5550 0    50   ~ 0
+RX
 $EndSCHEMATC
