File: Medidor/Medidor.sch (KiCad schematic (older format))
At the start: 47 parts, among them J1 TC2030-CTX-TAG_CONECT, SW1 Rotary_Encoder_Switch, SW2 SW_DPST_x2, U1 INA219-INA, U2 Serial, X1 32MHz

Commit message: Placement in progress
Parts:
- removed ANT1: 2450AT18D0100, symbol Device:Antenna
- removed Fil1: 2450FM07A0029T-medidor, symbol Medidor-rescue:2450FM07A0029T-medidor
- removed R4, R5: 1kΩ, Resistor_SMD:R_0402_1005Metric, symbol Device:R_Small_US
- added Fil1: 2450FM07A0029T, Medidor:baloon, symbol medidor:2450FM07A0029T
- added U3: 2450AT18D0100, Medidor:2450AT18D0100, symbol medidor:2450AT18D0100
- R1: footprint (none) -> Resistor_SMD:R_0805_2012Metric
- SW2: footprint (none) -> Medidor:botao
- U2: footprint (none) -> Connector:FanPinHeader_1x03_P2.54mm_Vertical
- X1: footprint (none) -> Medidor:cristal
Connections:
- net labels added: RC1, RC2, RC3
- net labels removed: AIN0, AIN1, R_B
- wire segments 188 -> 191
- no-connect marks 27 -> 26
Other:
- moved on the sheet: R8
Changed lines of the file:
@@
 F 0 "X1" V 7650 3800 50  0000 L CNN
 F 1 "32MHz" V 7850 3650 50  0000 L CNN
-F 2 "" H 7750 3950 50  0001 C CNN
+F 2 "Medidor:cristal" H 7750 3950 50  0001 C CNN
 F 3 "~" H 7750 3950 50  0001 C CNN
 	1    7750 3950
@@
 NoConn ~ 4750 3950
 NoConn ~ 4750 4050
-NoConn ~ 4750 4350
 NoConn ~ 4750 4450
 NoConn ~ 4750 4650
@@
 F 0 "R1" H 10250 1800 50  0000 C CNN
 F 1 "Shunt" H 10200 2000 50  0000 C CNN
-F 2 "" H 10350 1900 50  0001 C CNN
+F 2 "Resistor_SMD:R_0805_2012Metric" H 10350 1900 50  0001 C CNN
 F 3 "~" H 10350 1900 50  0001 C CNN
 	1    10350 1900
@@
 	8700 1850 7700 1850
 Connection ~ 7700 1850
-$Comp
-L Device:R_Small_US R4
-U 1 1 5D51C510
-P 7150 2300
-F 0 "R4" V 7200 2450 50  0000 C CNN
-F 1 "1kΩ" V 7200 2150 50  0000 C CNN
-F 2 "Resistor_SMD:R_0402_1005Metric" H 7150 2300 50  0001 C CNN
-F 3 "~" H 7150 2300 50  0001 C CNN
-	1    7150 2300
-	0    -1   -1   0
-$EndComp
-$Comp
-L Device:R_Small_US R5
-U 1 1 5D520673
-P 6800 1650
-F 0 "R5" V 6850 1800 50  0000 C CNN
-F 1 "1kΩ" V 6850 1500 50  0000 C CNN
-F 2 "Resistor_SMD:R_0402_1005Metric" H 6800 1650 50  0001 C CNN
-F 3 "~" H 6800 1650 50  0001 C CNN
-	1    6800 1650
-	0    -1   -1   0
-$EndComp
 Wire Wire Line
 	8700 2050 7550 2050
@@
 Text GLabel 8000 5600 0    50   Input ~ 0
 Ant
-$Comp
-L power:Earth #PWR0112
-U 1 1 5D328A7E
-P 10000 6000
-F 0 "#PWR0112" H 10000 5750 50  0001 C CNN
-F 1 "Earth" H 10000 5850 50  0001 C CNN
-F 2 "" H 10000 6000 50  0001 C CNN
-F 3 "~" H 10000 6000 50  0001 C CNN
-	1    10000 6000
-	1    0    0    -1
-$EndComp
-Connection ~ 10000 5600
-$Comp
-L Device:Antenna ANT1
-U 1 1 5D3263EB
-P 10000 5400
-F 0 "ANT1" H 10080 5389 50  0000 L CNN
-F 1 " 2450AT18D0100" H 10080 5298 50  0000 L CNN
-F 2 "" H 10000 5400 50  0001 C CNN
-F 3 "~" H 10000 5400 50  0001 C CNN
-	1    10000 5400
-	1    0    0    -1
-$EndComp
 Text Label 9650 5600 0    50   ~ 0
 RF
@@
 	6600 1700 6600 1650
 Wire Wire Line
-	6600 1650 6700 1650
-Wire Wire Line
-	6900 1650 7050 1650
-Wire Wire Line
 	7050 1650 7050 1950
 Wire Wire Line
 	7050 1950 8700 1950
 Wire Wire Line
-	7250 2300 7550 2300
-Wire Wire Line
 	7550 2050 7550 2300
-Wire Wire Line
-	6900 2300 7050 2300
 $Comp
 L Device:R_Small_US R7
@@
 Wire Wire Line
 	9000 6050 9000 5950
-Wire Wire Line
-	9500 5600 10000 5600
-$Comp
-L Device:R_Small_US R8
-U 1 1 5D3EB97D
-P 10000 5800
-F 0 "R8" H 10050 5950 50  0000 C CNN
-F 1 "NC" H 10050 5650 50  0000 C CNN
-F 2 "Resistor_SMD:R_0402_1005Metric" H 10000 5800 50  0001 C CNN
-F 3 "~" H 10000 5800 50  0001 C CNN
-	1    10000 5800
-	1    0    0    -1
-$EndComp
-Wire Wire Line
-	10000 5600 10000 5700
-Wire Wire Line
-	10000 6000 10000 5900
 $Comp
 L Device:C_Small C13
@@
 F 0 "SW2" H 5850 6193 50  0001 C CNN
 F 1 "SW_DPST_x2" H 5850 6194 50  0001 C CNN
-F 2 "" H 5850 6050 50  0001 C CNN
+F 2 "Medidor:botao" H 5850 6050 50  0001 C CNN
 F 3 "~" H 5850 6050 50  0001 C CNN
 	1    5850 6050
@@
 Wire Wire Line
 	2000 5500 2000 5400
-Text GLabel 4200 4150 0    50   Input ~ 0
-AIN0
+Text GLabel 4200 4350 0    50   Input ~ 0
+RC1
 Wire Wire Line
 	4200 4150 4750 4150
 Text GLabel 4200 4250 0    50   Input ~ 0
-AIN1
+RC2
 Wire Wire Line
 	4200 4250 4750 4250
 Text GLabel 1000 5450 0    50   Input ~ 0
-AIN1
+RC1
 Wire Wire Line
 	3100 5450 2800 5450
@@
 	1000 5450 1250 5450
 Text GLabel 3100 5450 2    50   Input ~ 0
-AIN0
+RC2
 $Comp
 L Device:R_Small_US R13
@@
 F 3 "" H 4650 6050 50  0001 C CNN
 	1    5650 4400
-	1    0    0    -1
-$EndComp
-$Comp
-L Medidor-rescue:2450FM07A0029T-medidor Fil1
-U 1 1 5D5CC96B
-P 8500 5600
-F 0 "Fil1" H 8750 5800 50  0000 L CNN
-F 1 "2450FM07A0029T-medidor" H 7900 5150 50  0000 L CNN
-F 2 "" H 8500 5600 50  0001 C CNN
-F 3 "" H 8500 5600 50  0001 C CNN
-	1    8500 5600
 	1    0    0    -1
 $EndComp
@@
 	3250 6250 700  6250
 Wire Notes Line
-	7600 5100 10750 5100
-Wire Notes Line
-	10750 5100 10750 6250
-Wire Notes Line
-	10750 6250 7600 6250
+	11150 5100 11150 6250
 Wire Notes Line
 	7600 6250 7600 5100
@@
 	1900 4450 2200 4450
 Connection ~ 1900 4650
-Text Label 2200 4450 0    50   ~ 0
-R_B
 $Comp
 L Medidor-rescue:Serial-medidor U2
@@
 F 0 "U2" V 4196 7278 50  0000 L CNN
 F 1 "Serial" V 4287 7278 50  0000 L CNN
-F 2 "" H 4300 7050 50  0001 C CNN
+F 2 "Connector:FanPinHeader_1x03_P2.54mm_Vertical" H 4300 7050 50  0001 C CNN
 F 3 "" H 4300 7050 50  0001 C CNN
 	1    4300 7050
@@
 Text Label 5400 5550 0    50   ~ 0
 RX
+Text GLabel 2200 4450 2    50   Input ~ 0
+RC3
+Text GLabel 4200 4150 0    50   Input ~ 0
+RC3
+Wire Wire Line
+	4200 4350 4750 4350
+Wire Notes Line
+	7600 5100 11150 5100
+Wire Notes Line
+	7600 6250 11150 6250
+$Comp
+L power:Earth #PWR0112
+U 1 1 5D328A7E
+P 9800 6100
+F 0 "#PWR0112" H 9800 5850 50  0001 C CNN
+F 1 "Earth" H 9800 5950 50  0001 C CNN
+F 2 "" H 9800 6100 50  0001 C CNN
+F 3 "~" H 9800 6100 50  0001 C CNN
+	1    9800 6100
+	1    0    0    -1
+$EndComp
+Wire Wire Line
+	9500 5600 9800 5600
+$Comp
+L medidor:2450AT18D0100 U3
+U 1 1 5D426326
+P 10250 5700
+F 0 "U3" H 10275 6015 50  0001 C CNN
+F 1 "2450AT18D0100" H 10275 5427 50  0000 C CNN
+F 2 "Medidor:2450AT18D0100" H 10250 5600 50  0001 C CNN
+F 3 "" H 10250 5600 50  0001 C CNN
+	1    10250 5700
+	1    0    0    1
+$EndComp
+Wire Wire Line
+	9800 5750 9800 5850
+Wire Wire Line
+	9800 6100 9800 6050
+$Comp
+L Device:R_Small_US R8
+U 1 1 5D3EB97D
+P 9800 5950
+F 0 "R8" H 9850 6100 50  0000 C CNN
+F 1 "NC" H 9850 5800 50  0000 C CNN
+F 2 "Resistor_SMD:R_0402_1005Metric" H 9800 5950 50  0001 C CNN
+F 3 "~" H 9800 5950 50  0001 C CNN
+	1    9800 5950
+	1    0    0    -1
+$EndComp
+$Comp
+L power:Earth #PWR0153
+U 1 1 5D517F43
+P 11000 5650
+F 0 "#PWR0153" H 11000 5400 50  0001 C CNN
+F 1 "Earth" H 11000 5500 50  0001 C CNN
+F 2 "" H 11000 5650 50  0001 C CNN
+F 3 "~" H 11000 5650 50  0001 C CNN
+	1    11000 5650
+	1    0    0    -1
+$EndComp
+Wire Wire Line
+	11000 5650 11000 5600
+Wire Wire Line
+	11000 5600 10750 5600
+$Comp
+L power:Earth #PWR0154
+U 1 1 5D52397E
+P 10800 5850
+F 0 "#PWR0154" H 10800 5600 50  0001 C CNN
+F 1 "Earth" H 10800 5700 50  0001 C CNN
+F 2 "" H 10800 5850 50  0001 C CNN
+F 3 "~" H 10800 5850 50  0001 C CNN
+	1    10800 5850
+	1    0    0    -1
+$EndComp
+Wire Wire Line
+	10800 5850 10800 5750
+Wire Wire Line
+	10800 5750 10750 5750
+$Comp
+L medidor:2450FM07A0029T Fil1
+U 1 1 5D577615
+P 8500 5600
+F 0 "Fil1" H 8894 5621 50  0000 L CNN
+F 1 "2450FM07A0029T" H 8894 5530 50  0000 L CNN
+F 2 "Medidor:baloon" H 8500 5600 50  0001 C CNN
+F 3 "" H 8500 5600 50  0001 C CNN
+	1    8500 5600
+	1    0    0    -1
+$EndComp
+Wire Wire Line
+	6600 1650 7050 1650
+Wire Wire Line
+	6900 2300 7550 2300
 $EndSCHEMATC

Commit message: Replacement
Parts:
- removed U2: Serial, Connector:FanPinHeader_1x03_P2.54mm_Vertical, symbol Medidor-rescue:Serial-medidor
- added U2: Serial, symbol medidor:Serial
- R7: value 1k -> 0
Connections:
- net Earth is gone; now on net GND: C1.1, C10.1, C11.1, C12.2, C13.2, C14.2, C15.2, C16.2, C2.1, C3.1, C4.1, C7.1, C8.1, C9.1, Display1.1 (GND), Fil1.2 (GND), Fil1.4 (GND), J1.5 (GND), MCU1.31 (VSS), MCU1.45 (VSS), MCU1.49 (VSS), R6.2, R8.2, SW1.C, SW1.S2, SW2.1 (A), U1.3 (GND), U1.7 (A0), U1.8 (A1), U3.2 (GND), U3.3 (GND), US1.5 (GND), dc1.2 (GND), dc1.3 (GND), dc1.6 (GND), dc1.7 (GND)
- net RF: now also R8.1
- net RX: now also U2.3 (Rx)
- net TX: now also U2.2 (Tx)
- net GND: now reaches U3.4 (GND)
- net GND: now also U2.1 (GND); no longer R8.1
Other:
- moved on the sheet: R8

Commit message: more replacement
Parts:
- Fil1: symbol medidor:2450FM07A0029T -> Medidor-rescue:2450FM07A0029T-medidor
- U2: symbol medidor:Serial -> Medidor-rescue:Serial-medidor
- U3: symbol medidor:2450AT18D0100 -> Medidor-rescue:2450AT18D0100-medidor
Changed lines of the file:
@@
 	10800 5750 10750 5750
 $Comp
-L medidor:2450FM07A0029T Fil1
+L Medidor-rescue:2450FM07A0029T-medidor Fil1
 U 1 1 5D577615
 P 8500 5600
@@
 $EndComp
 $Comp
-L medidor:2450AT18D0100 U3
+L Medidor-rescue:2450AT18D0100-medidor U3
 U 1 1 5D426326
 P 10250 5700
@@
 	2450 5450 2800 5450
 $Comp
-L medidor:Serial U2
+L Medidor-rescue:Serial-medidor U2
 U 1 1 5D480BDF
 P 4300 7050

Commit message: Add files via upload
Parts:
- added U10, U7, U8, U9: spacer, Medidor:spacer, symbol Medidor-rescue:spacer-medidor
- added U4, U5, U6: Fiducial, Fiducial:Fiducial_0.75mm_Mask1.5mm, symbol Medidor-rescue:Fiducial-medidor
Connections:
- net LEDMCU: now also MCU1.42 (P0.30/AIN6); no longer MCU1.8 (P0.06)
- net RC1: now also MCU1.38 (P0.26); no longer MCU1.6 (P0.04/AIN2)
- net RC2: now also MCU1.39 (P0.27); no longer MCU1.5 (P0.03/AIN1)
- net RC3: now also MCU1.43 (P0.31/AIN7); no longer MCU1.4 (P0.02/AIN0)
- net RX: now also MCU1.4 (P0.02/AIN0); no longer MCU1.16 (P0.13)
- net SCL: now also MCU1.9 (P0.07); no longer MCU1.43 (P0.31/AIN7)
- net SDA: now also MCU1.8 (P0.06); no longer MCU1.42 (P0.30/AIN6)
- net TX: now also MCU1.3 (P0.01/XL2); no longer MCU1.15 (P0.12)
Changed lines of the file:
@@
 Wire Wire Line
 	5400 2500 5400 3550
-Text GLabel 5750 3050 2    50   Input ~ 0
+Text GLabel 4250 4550 0    50   Input ~ 0
 SDA
 Wire Wire Line
@@
 Wire Wire Line
 	5700 3050 5750 3050
-Text GLabel 5750 2900 2    50   Input ~ 0
+Text GLabel 4250 4650 0    50   Input ~ 0
 SCL
 Wire Wire Line
@@
 Wire Wire Line
 	3800 1400 3800 1550
-Text GLabel 4250 4550 0    50   Input ~ 0
+Text GLabel 5750 3050 2    50   Input ~ 0
 LEDMCU
 Wire Wire Line
@@
 ALIMENTAÇÂO
 NoConn ~ 4750 3950
-NoConn ~ 4750 4050
 NoConn ~ 4750 4450
-NoConn ~ 4750 4650
 NoConn ~ 4750 4750
 NoConn ~ 4750 4850
@@
 Wire Wire Line
 	2000 5500 2000 5400
-Text GLabel 4200 4350 0    50   Input ~ 0
+Text GLabel 6100 3350 2    50   Input ~ 0
 RC1
-Wire Wire Line
-	4200 4150 4750 4150
-Text GLabel 4200 4250 0    50   Input ~ 0
+Text GLabel 6050 3200 2    50   Input ~ 0
 RC2
-Wire Wire Line
-	4200 4250 4750 4250
 Text GLabel 1000 5450 0    50   Input ~ 0
 RC1
@@
 	3000 600  3000 2200
 Wire Notes Line
-	3000 2200 4500 2200
-Wire Notes Line
 	4500 2200 4500 600
 Wire Notes Line
@@
 NoConn ~ 5200 5350
 Wire Wire Line
-	5300 5550 5300 5350
-Wire Wire Line
 	4300 6600 4200 6600
 Wire Wire Line
@@
 Wire Wire Line
 	9800 2050 10000 2050
-NoConn ~ 6100 3550
-NoConn ~ 6000 3550
 Wire Wire Line
 	1900 4650 1900 4450
@@
 Text Label 4500 6600 0    50   ~ 0
 RX
-Text Label 5300 5550 0    50   ~ 0
+Text Label 4650 4050 0    50   ~ 0
 TX
-Wire Wire Line
-	5400 5350 5400 5550
-Text Label 5400 5550 0    50   ~ 0
+Text Label 4650 4150 0    50   ~ 0
 RX
 Text GLabel 2200 4450 2    50   Input ~ 0
 RC3
-Text GLabel 4200 4150 0    50   Input ~ 0
+Text GLabel 5750 2900 2    50   Input ~ 0
 RC3
-Wire Wire Line
-	4200 4350 4750 4350
 Wire Notes Line
 	7600 5100 11150 5100
@@
 	1    0    0    -1
 $EndComp
+Wire Notes Line
+	3000 2200 4500 2200
+$Comp
+L Medidor-rescue:Fiducial-medidor U4
+U 1 1 5D438E8C
+P 9350 3200
+F 0 "U4" H 9584 3246 50  0000 L CNN
+F 1 "Fiducial" H 9584 3155 50  0000 L CNN
+F 2 "Fiducial:Fiducial_0.75mm_Mask1.5mm" H 9350 3250 50  0001 C CNN
+F 3 "" H 9350 3250 50  0001 C CNN
+	1    9350 3200
+	1    0    0    -1
+$EndComp
+$Comp
+L Medidor-rescue:Fiducial-medidor U6
+U 1 1 5D43A2B9
+P 10300 3200
+F 0 "U6" H 10534 3246 50  0000 L CNN
+F 1 "Fiducial" H 10534 3155 50  0000 L CNN
+F 2 "Fiducial:Fiducial_0.75mm_Mask1.5mm" H 10300 3250 50  0001 C CNN
+F 3 "" H 10300 3250 50  0001 C CNN
+	1    10300 3200
+	1    0    0    -1
+$EndComp
+$Comp
+L Medidor-rescue:Fiducial-medidor U5
+U 1 1 5D43A693
+P 9800 3600
+F 0 "U5" H 10034 3646 50  0000 L CNN
+F 1 "Fiducial" H 10034 3555 50  0000 L CNN
+F 2 "Fiducial:Fiducial_0.75mm_Mask1.5mm" H 9800 3650 50  0001 C CNN
+F 3 "" H 9800 3650 50  0001 C CNN
+	1    9800 3600
+	1    0    0    -1
+$EndComp
+$Comp
+L Medidor-rescue:spacer-medidor U7
+U 1 1 5D43D50E
+P 9650 4100
+F 0 "U7" H 9819 4146 50  0000 L CNN
+F 1 "spacer" H 9819 4055 50  0000 L CNN
+F 2 "Medidor:spacer" H 9650 4100 50  0001 C CNN
+F 3 "" H 9650 4100 50  0001 C CNN
+	1    9650 4100
+	1    0    0    -1
+$EndComp
+$Comp
+L Medidor-rescue:spacer-medidor U9
+U 1 1 5D43E3DB
+P 10350 4100
+F 0 "U9" H 10519 4146 50  0000 L CNN
+F 1 "spacer" H 10519 4055 50  0000 L CNN
+F 2 "Medidor:spacer" H 10350 4100 50  0001 C CNN
+F 3 "" H 10350 4100 50  0001 C CNN
+	1    10350 4100
+	1    0    0    -1
+$EndComp
+$Comp
+L Medidor-rescue:spacer-medidor U8
+U 1 1 5D43E795
+P 10000 4500
+F 0 "U8" H 10169 4546 50  0000 L CNN
+F 1 "spacer" H 10169 4455 50  0000 L CNN
+F 2 "Medidor:spacer" H 10000 4500 50  0001 C CNN
+F 3 "" H 10000 4500 50  0001 C CNN
+	1    10000 4500
+	1    0    0    -1
+$EndComp
+$Comp
+L Medidor-rescue:spacer-medidor U10
+U 1 1 5D44398C
+P 9400 4550
+F 0 "U10" H 9569 4596 50  0000 L CNN
+F 1 "spacer" H 9569 4505 50  0000 L CNN
+F 2 "Medidor:spacer" H 9400 4550 50  0001 C CNN
+F 3 "" H 9400 4550 50  0001 C CNN
+	1    9400 4550
+	1    0    0    -1
+$EndComp
+Wire Wire Line
+	4250 4650 4750 4650
+Wire Wire Line
+	6050 3200 6000 3200
+Wire Wire Line
+	6000 3200 6000 3550
+Wire Wire Line
+	6100 3550 6100 3350
+NoConn ~ 4750 4250
+NoConn ~ 4750 4350
+Wire Wire Line
+	4750 4050 4650 4050
+Wire Wire Line
+	4750 4150 4650 4150
+NoConn ~ 5400 5350
+NoConn ~ 5300 5350
 $EndSCHEMATC

Commit message: conexões
Connections:
- net LEDMCU: now also MCU1.43 (P0.31/AIN7); no longer MCU1.42 (P0.30/AIN6)
- net RC1: now also MCU1.42 (P0.30/AIN6); no longer MCU1.38 (P0.26)
- net RC3: now also MCU1.38 (P0.26); no longer MCU1.43 (P0.31/AIN7)
Changed lines of the file:
@@
 Wire Wire Line
 	3800 1400 3800 1550
-Text GLabel 5750 3050 2    50   Input ~ 0
+Text GLabel 5750 2900 2    50   Input ~ 0
 LEDMCU
 Wire Wire Line
@@
 Wire Wire Line
 	2000 5500 2000 5400
-Text GLabel 6100 3350 2    50   Input ~ 0
+Text GLabel 5750 3050 2    50   Input ~ 0
 RC1
 Text GLabel 6050 3200 2    50   Input ~ 0
@@
 Text GLabel 2200 4450 2    50   Input ~ 0
 RC3
-Text GLabel 5750 2900 2    50   Input ~ 0
+Text GLabel 6100 3350 2    50   Input ~ 0
 RC3
 Wire Notes Line

Commit message: Footprints USB, DISPLAY, INA219 E L78L associados
Parts:
- U1: footprint Package_TO_SOT_SMD:SuperSOT-8 -> Medidor:INA219
- US1: footprint (none) -> Connector_USB:USB_Micro-B_Wuerth_629105150521_CircularHoles
- dc1: footprint Package_TO_SOT_SMD:SuperSOT-8 -> Medidor:L78L
Changed lines of the file:
@@
 F 0 "dc1" H 2225 7533 50  0001 C CNN
 F 1 "DC-DC" H 2225 7533 50  0000 C CNN
-F 2 "Package_TO_SOT_SMD:SuperSOT-8" H 2200 7300 50  0001 C CNN
+F 2 "Medidor:L78L" H 2200 7300 50  0001 C CNN
 F 3 "" H 2200 7300 50  0001 C CNN
 	1    2200 7300
@@
 F 0 "US1" H 908 7675 50  0000 C CNN
 F 1 "USB" H 908 7584 50  0000 C CNN
-F 2 "" H 850 7300 50  0001 C CNN
+F 2 "Connector_USB:USB_Micro-B_Wuerth_629105150521_CircularHoles" H 850 7300 50  0001 C CNN
 F 3 "" H 850 7300 50  0001 C CNN
 	1    850  7250
@@
 F 0 "U1" H 9200 2717 50  0000 C CNN
 F 1 "INA219-INA" H 9200 2626 50  0000 C CNN
-F 2 "Package_TO_SOT_SMD:SuperSOT-8" H 9200 1850 50  0001 L BNN
+F 2 "Medidor:INA219" H 9200 1850 50  0001 L BNN
 F 3 "" H 9200 1850 50  0001 L BNN
 F 4 "SOT-23-8 Texas Instruments" H 9200 1850 50  0001 L BNN "Campo4"

Commit message: replacement again and again and again
Parts:
- U2: footprint (none) -> Connector_PinHeader_2.54mm:PinHeader_1x03_P2.54mm_Vertical
Connections:
- net GND: now also SW2.2 (B); no longer SW2.1 (A)
- net LEDMCU: now also MCU1.20 (P0.17); no longer MCU1.43 (P0.31/AIN7)
- net RC1: now also MCU1.16 (P0.13); no longer MCU1.42 (P0.30/AIN6)
- net RC2: now also MCU1.15 (P0.12); no longer MCU1.39 (P0.27)
- net RC3: now also MCU1.14 (P0.11); no longer MCU1.38 (P0.26)
- net nRESET: now also SW2.1 (A); no longer SW2.2 (B)
Changed lines of the file:
@@
 Text GLabel 4250 4550 0    50   Input ~ 0
 SDA
-Wire Wire Line
-	5700 3550 5700 3050
-Wire Wire Line
-	5700 3050 5750 3050
 Text GLabel 4250 4650 0    50   Input ~ 0
 SCL
-Wire Wire Line
-	5750 2900 5600 2900
-Wire Wire Line
-	5600 2900 5600 3550
 NoConn ~ 5800 3550
 NoConn ~ 6200 3550
@@
 NoConn ~ 6000 5350
 NoConn ~ 5900 5350
-NoConn ~ 5800 5350
 NoConn ~ 5700 5350
 NoConn ~ 5600 5350
@@
 Wire Wire Line
 	3800 1400 3800 1550
-Text GLabel 5750 2900 2    50   Input ~ 0
+Text GLabel 5800 5650 0    50   Input ~ 0
 LEDMCU
 Wire Wire Line
@@
 L Switch:SW_DPST_x2 SW2
 U 1 1 5D49EA8B
-P 5850 6050
-F 0 "SW2" H 5850 6193 50  0001 C CNN
-F 1 "SW_DPST_x2" H 5850 6194 50  0001 C CNN
-F 2 "Medidor:botao" H 5850 6050 50  0001 C CNN
-F 3 "~" H 5850 6050 50  0001 C CNN
-	1    5850 6050
-	1    0    0    -1
-$EndComp
-Wire Wire Line
-	5600 6050 5650 6050
-Wire Wire Line
-	6050 6050 6200 6050
+P 6400 6050
+F 0 "SW2" H 6400 6193 50  0001 C CNN
+F 1 "SW_DPST_x2" H 6400 6194 50  0001 C CNN
+F 2 "Medidor:botao" H 6400 6050 50  0001 C CNN
+F 3 "~" H 6400 6050 50  0001 C CNN
+	1    6400 6050
+	1    0    0    -1
+$EndComp
 Wire Wire Line
 	6200 6050 6200 5500
 Connection ~ 6200 5500
-Wire Wire Line
-	5600 6150 5600 6050
 $Comp
 L Device:R_Small_US R9
@@
 Wire Wire Line
 	2000 5500 2000 5400
-Text GLabel 5750 3050 2    50   Input ~ 0
+Text GLabel 5200 6050 0    50   Input ~ 0
 RC1
-Text GLabel 6050 3200 2    50   Input ~ 0
+Text GLabel 5200 5900 0    50   Input ~ 0
 RC2
 Text GLabel 1000 5450 0    50   Input ~ 0
@@
 Wire Wire Line
 	3950 6800 3950 7000
-NoConn ~ 5200 5350
 Wire Wire Line
 	4300 6600 4200 6600
@@
 Text GLabel 2200 4450 2    50   Input ~ 0
 RC3
-Text GLabel 6100 3350 2    50   Input ~ 0
+Text GLabel 5200 5750 0    50   Input ~ 0
 RC3
 Wire Notes Line
@@
 L power:GND #PWR0111
 U 1 1 5D44E86B
-P 5600 6150
-F 0 "#PWR0111" H 5600 5900 50  0001 C CNN
-F 1 "GND" H 5600 6000 50  0000 C CNN
-F 2 "" H 5600 6150 50  0001 C CNN
-F 3 "" H 5600 6150 50  0001 C CNN
-	1    5600 6150
+P 6650 6100
+F 0 "#PWR0111" H 6650 5850 50  0001 C CNN
+F 1 "GND" H 6650 5950 50  0000 C CNN
+F 2 "" H 6650 6100 50  0001 C CNN
+F 3 "" H 6650 6100 50  0001 C CNN
+	1    6650 6100
 	1    0    0    -1
 $EndComp
@@
 F 0 "U2" V 4196 7278 50  0001 L CNN
 F 1 "Serial" V 4242 7278 50  0000 L CNN
-F 2 "" H 4300 7050 50  0001 C CNN
+F 2 "Connector_PinHeader_2.54mm:PinHeader_1x03_P2.54mm_Vertical" H 4300 7050 50  0001 C CNN
 F 3 "" H 4300 7050 50  0001 C CNN
 	1    4300 7050
@@
 Wire Wire Line
 	4250 4650 4750 4650
-Wire Wire Line
-	6050 3200 6000 3200
-Wire Wire Line
-	6000 3200 6000 3550
-Wire Wire Line
-	6100 3550 6100 3350
 NoConn ~ 4750 4250
 NoConn ~ 4750 4350
@@
 Wire Wire Line
 	4750 4150 4650 4150
-NoConn ~ 5400 5350
-NoConn ~ 5300 5350
+Wire Wire Line
+	5200 5350 5200 5750
+Wire Wire Line
+	5200 5900 5300 5900
+Wire Wire Line
+	5300 5900 5300 5350
+Wire Wire Line
+	5200 6050 5400 6050
+Wire Wire Line
+	5400 6050 5400 5350
+Wire Wire Line
+	6650 6100 6650 6050
+Wire Wire Line
+	6650 6050 6600 6050
+Wire Wire Line
+	5800 5650 5800 5350
+NoConn ~ 6100 3550
+NoConn ~ 6000 3550
+NoConn ~ 5700 3550
+NoConn ~ 5600 3550
 $EndSCHEMATC

Commit message: bonito
Connections:
- net RX: now also U2.2 (Tx); no longer U2.3 (Rx)
- net TX: now also U2.3 (Rx); no longer U2.2 (Tx)
Changed lines of the file:
@@
 Wire Wire Line
 	4300 6600 4300 6800
+Text Label 4500 6600 0    50   ~ 0
+TX
 Text Label 4200 6600 0    50   ~ 0
-TX
-Text Label 4500 6600 0    50   ~ 0
 RX
 Text Label 4650 4050 0    50   ~ 0
