File: Medidor/Medidor.kicad_pcb (KiCad board)
At the start: 2 copper layers, 59.9 x 47.1 mm, 52 parts, among them J1 TC2030-CTX-TAG_CONECT, SW1 Rotary_Encoder_Switch, SW2 SW_DPST_x2, U1 INA219-INA, U10 spacer, U2 Serial, U3 2450AT18D0100, U4 Fiducial, U5 Fiducial, U6 Fiducial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

Commit message: Ligações feitas
Parts:
- US1: moved to F.Cu
- moved SW2 0.59 mm to (92.2, 120.1)
- moved Display1 0.57 mm to (126.4, 89.2)
- moved J1 0.14 mm to (105.5, 101.8)
- turned US1 to 270 degrees
Routing:
- net +3V3: track 98.4 -> 111.4 mm, vias 31 -> 32
- net (no net): track 14.3 -> 5.44 mm, vias 8 -> 12
- net +5V: track 0.00 -> 2.67 mm, vias 5 -> 0
- net SDA: track 26.7 -> 29.3 mm
- net SWDIO: track 16.1 -> 14.1 mm
- net GND: track 23.3 -> 25.2 mm, vias 293 -> 285
- net SCL: track 26.0 -> 27.6 mm
- net nRESET: track 21.0 -> 21.7 mm
- net Net-(C5-Pad2): track 2.13 -> 2.84 mm
- net Net-(C5-Pad1): track 2.22 -> 2.77 mm
- removed copper zone on B.Cu, net +5V

Commit message: replacement again and again and again
Parts:
- moved U2 55.1 mm to (92.2, 92.2), turned to 0 degrees
- moved US1 55.0 mm to (139.4, 116.6), turned to 90 degrees
- moved U3 54.2 mm to (132.7, 90.2), turned to 0 degrees
- moved C16 54.1 mm to (138.4, 125.1)
- moved R8 49.4 mm to (132.5, 93.2), turned to 180 degrees
- moved R7 47.3 mm to (133.0, 94.8), turned to 90 degrees
- moved Screw_Terminal 47.0 mm to (90.4, 101.6)
- moved R6 44.5 mm to (132.5, 96.8), turned to 180 degrees
- moved C12 41.5 mm to (131.6, 112.5)
- moved dc1 41.1 mm to (131.3, 120.0), turned to 180 degrees
- moved R1 39.6 mm to (94.7, 103.9), turned to 90 degrees
- moved R15 36.0 mm to (96.5, 103.5), turned to 0 degrees
- moved R16 35.6 mm to (96.5, 104.5), turned to 0 degrees
- moved C11 33.4 mm to (98.8, 108.5), turned to 0 degrees
- moved J1 33.1 mm to (138.0, 107.9)
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Connections:
- MCU1 pad 14: Net-(MCU1-Pad14) -> RC3
- MCU1 pad 15: Net-(MCU1-Pad15) -> RC2
- MCU1 pad 16: Net-(MCU1-Pad16) -> RC1
- MCU1 pad 20: Net-(MCU1-Pad20) -> LEDMCU
- MCU1 pad 38: RC3 -> Net-(MCU1-Pad38)
- MCU1 pad 39: RC2 -> Net-(MCU1-Pad39)
- MCU1 pad 42: RC1 -> Net-(MCU1-Pad42)
- MCU1 pad 43: LEDMCU -> Net-(MCU1-Pad43)
- SW2 pad 1: GND -> nRESET
- SW2 pad 2: nRESET -> GND
Routing:
- net +3V3: track 111.4 -> 0.00 mm, vias 32 -> 0
- net RC2: track 34.0 -> 0.00 mm
- net SDA: track 29.3 -> 0.00 mm, vias 2 -> 0
- net SCL: track 27.6 -> 0.00 mm
- net RC1: track 27.4 -> 0.00 mm
- net /TX: track 26.5 -> 0.00 mm
- net GND: track 25.2 -> 0.00 mm, vias 285 -> 0
- net /RX: track 24.4 -> 0.00 mm
- net RC3: track 23.6 -> 0.00 mm
- net LEDMCU: track 22.9 -> 0.00 mm, vias 2 -> 0
- net nRESET: track 21.7 -> 0.00 mm, vias 5 -> 0
- net Net-(Fil1-Pad3): track 19.7 -> 0.00 mm
- net SWDIO: track 14.1 -> 0.00 mm
- net SWDCLK: track 12.2 -> 0.00 mm
- net Net-(C3-Pad2): track 8.18 -> 0.00 mm
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- removed copper zone on B.Cu, net +3V3
- removed copper zone on F.Cu, net +3V3
- removed copper zone on F.Cu, net +5V
- removed copper zone on B.Cu, net GND
- removed copper zone on F.Cu, net GND

Commit message: bonito
Parts:
- moved U3 20.6 mm to (141.6, 108.8), turned to 270 degrees
- moved R8 17.6 mm to (142.2, 107.8), turned to 0 degrees
- moved R7 14.5 mm to (141.7, 106.4), turned to 270 degrees
- moved R6 12.7 mm to (142.2, 105.0), turned to 0 degrees
- moved SW2 6.82 mm to (126.6, 124.1), turned to 270 degrees
- moved J1 6.42 mm to (131.7, 108.8), turned to 180 degrees
- moved C16 6.10 mm to (132.8, 127.4), turned to 180 degrees
- moved R13 6.08 mm to (121.8, 117.7), turned to 90 degrees
- moved R14 5.90 mm to (103.9, 129.9)
- moved D1 5.28 mm to (120.2, 117.2), turned to 270 degrees
- moved R11 4.24 mm to (113.8, 129.8), turned to 90 degrees
- moved C15 3.30 mm to (112.5, 127.7), turned to 90 degrees
- moved SW1 3.30 mm to (116.2, 124.3)
- moved US1 2.60 mm to (139.4, 119.3)
- moved C12 2.16 mm to (131.8, 114.6)
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Connections:
- U2 pad 2: /TX -> /RX
- U2 pad 3: /RX -> /TX
Routing:
- net +3V3: track 0.00 -> 185.8 mm, vias 0 -> 20
- net nRESET: track 0.00 -> 32.0 mm, vias 0 -> 3
- net RC3: track 0.00 -> 31.3 mm
- net SCL: track 0.00 -> 29.4 mm, vias 0 -> 2
- net RC2: track 0.00 -> 29.1 mm
- net SDA: track 0.00 -> 27.4 mm
- net /RX: track 0.00 -> 26.9 mm, vias 0 -> 2
- net /TX: track 0.00 -> 23.6 mm, vias 0 -> 2
- net RC1: track 0.00 -> 19.7 mm
- net Net-(Fil1-Pad3): track 0.00 -> 17.3 mm
- net SWDIO: track 0.00 -> 16.7 mm
- net SWDCLK: track 0.00 -> 12.3 mm
- net LEDMCU: track 0.00 -> 10.3 mm
- net +5V: track 0.00 -> 9.63 mm
- net Net-(C1-Pad2): track 0.00 -> 8.18 mm
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- added copper zone on B.Cu, net +3V3
- added copper zone on F.Cu, net +3V3
- added copper zone on B.Cu, net GND
- added copper zone on F.Cu, net GND
- added copper zone on F.Cu, net Net-(R1-Pad1)
- added copper zone on F.Cu, net Net-(R1-Pad2)
Other:
- board size 59.9 x 47.1 mm -> 60 x 47.1 mm
- net class Suply: trace_width 0.4 -> 0.6
- board text added: "Rx"
- board text added: "Tx"

Commit message: Acabamento
Parts:
- removed Screw_Terminal: TerminalBlock_Altech_AK300-2_P5.00mm, TerminalBlock:TerminalBlock_Altech_AK300-2_P5.00mm
- removed U10, U7, U8, U9: spacer, Medidor:spacer
- added G***: LOGO, Medidor:multi1, F.Cu at (141.7, 99.9)
- added REF**: MountingHole_2.2mm_M2_Pad, MountingHole:MountingHole_2.2mm_M2_Pad, F.Cu at (140.6, 132.1)
- added REF**: MountingHole_2.2mm_M2_Pad, MountingHole:MountingHole_2.2mm_M2_Pad, F.Cu at (140.4, 91.2)
- added REF**: MountingHole_2.2mm_M2_Pad, MountingHole:MountingHole_2.2mm_M2_Pad, F.Cu at (86.8, 132.2)
- added REF**: MountingHole_2.2mm_M2_Pad, MountingHole:MountingHole_2.2mm_M2_Pad, F.Cu at (86.8, 91.4)
- added TER1: terminal-medidor, Medidor:Screw, F.Cu at (89.1, 101.5)
- D1, R13: moved to B.Cu
- U2: footprint Connector:FanPinHeader_1x03_P2.54mm_Vertical -> Connector_PinHeader_2.54mm:PinHeader_1x03_P2.54mm_Vertical
- moved U2 25.5 mm to (86.6, 117.1), turned to 180 degrees
- moved U4 5.30 mm to (136.7, 91.1)
- moved U5 4.83 mm to (137.1, 133.5)
- moved D1 3.06 mm to (120.0, 120.2)
- moved R13 2.74 mm to (121.8, 120.5)
- moved C14 2.67 mm to (111.8, 121.1)
- moved C15 2.67 mm to (109.9, 127.6)
- moved R10 2.67 mm to (111.7, 123.2)
- moved R12 2.67 mm to (111.1, 127.6)
- moved R14 2.67 mm to (101.2, 129.8)
- moved R9 2.67 mm to (110.3, 121.5)
- moved SW1 2.67 mm to (113.5, 124.2)
- moved R11 2.67 mm to (111.1, 129.7)
- moved R2 1.74 mm to (110.0, 106.4), turned to 0 degrees
- moved US1 1.74 mm to (139.4, 121.0)
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Connections:
- MCU1 pad 3: /TX -> Net-(MCU1-Pad3)
- MCU1 pad 4: /RX -> Net-(MCU1-Pad4)
- MCU1 pad 6: Net-(MCU1-Pad6) -> SDA
- MCU1 pad 7: Net-(MCU1-Pad7) -> SCL
- MCU1 pad 8: SDA -> /RX
- MCU1 pad 9: SCL -> /TX
Routing:
- net +3V3: track 185.8 -> 127.3 mm, vias 20 -> 25
- net SCL: track 29.4 -> 46.2 mm, vias 2 -> 0
- net /TX: track 23.6 -> 37.7 mm, vias 2 -> 0
- net GND: track 3.76 -> 13.9 mm, vias 783 -> 558
- net /RX: track 26.9 -> 36.8 mm, vias 2 -> 0
- net LEDMCU: track 10.3 -> 15.2 mm, vias 0 -> 1
- net SWDIO: track 16.7 -> 20.0 mm
- net RC1: track 19.7 -> 21.8 mm
- net +5V: track 9.63 -> 11.7 mm
- net Net-(L1-Pad1): track 3.04 -> 1.81 mm
- net SWDCLK: track 12.3 -> 13.4 mm
- net RC3: track 31.3 -> 32.5 mm
- net Net-(C3-Pad2): track 7.87 -> 6.94 mm
- net Net-(C2-Pad2): track 7.48 -> 6.73 mm
Other:
- board size 60 x 47.1 mm -> 60.1 x 47.1 mm
- net class Ant: via_dia 0.5 -> 0.6
- net class Default: via_dia 0.5 -> 0.6
- net class Suply: via_dia 0.8 -> 0.6; via_drill 0.5 -> 0.3
- board text added: "Meter One for All UFAL C.I. 2019.1 José Carlos Pinheiro Filho Glauber Braga Tatiane"

Commit message: acabamento 2
Parts:
- moved D1 4.26 mm to (118.3, 124.2)
- moved R13 3.58 mm to (120.0, 123.6)
- moved R1 0.06 mm to (94.2, 104.1)
Routing:
- net +3V3: track 127.3 -> 134.7 mm
- net LEDMCU: track 15.2 -> 18.1 mm
- net GND: track 13.9 -> 15.7 mm, vias 558 -> 556
- net Net-(R1-Pad1): track 2.10 -> 1.25 mm
- net Net-(R1-Pad2): track 2.10 -> 1.43 mm
Other:
- board text removed: "GND"

Commit message: acabamento 2.1
Routing:
- net GND: track 15.7 -> 18.3 mm, vias 556 -> 533
Changed lines of the file:
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@@
     (thickness 1.6)
     (drawings 22)
-    (tracks 843)
+    (tracks 826)
     (zones 0)
     (modules 53)
@@
   (segment (start 116.8745 103.451) (end 115.8462 103.451) (width 0.2) (layer F.Cu) (net 11))
   (segment (start 115.8462 103.451) (end 114.7508 104.5464) (width 0.2) (layer F.Cu) (net 11))
+  (segment (start 114.3508 89.1032) (end 112.9665 89.1032) (width 0.2) (layer F.Cu) (net 11))
   (segment (start 107.0864 108.7628) (end 109.3216 106.5276) (width 0.2) (layer F.Cu) (net 11))
-  (segment (start 103.886 107.95) (end 104.6988 108.7628) (width 0.2) (layer F.Cu) (net 11))
-  (segment (start 103.886 101.4984) (end 103.886 107.95) (width 0.2) (layer F.Cu) (net 11))
+  (segment (start 112.4712 89.662) (end 112.4712 92.9132) (width 0.2) (layer F.Cu) (net 11))
+  (segment (start 112.9665 89.1032) (end 112.4712 89.662) (width 0.2) (layer F.Cu) (net 11))
   (segment (start 112.4712 92.9132) (end 103.886 101.4984) (width 0.2) (layer F.Cu) (net 11))
-  (segment (start 115.544501 89.436501) (end 114.646001 89.436501) (width 0.2) (layer F.Cu) (net 11))
+  (segment (start 103.886 101.4984) (end 103.886 107.95) (width 0.2) (layer F.Cu) (net 11))
+  (segment (start 103.886 107.95) (end 104.6988 108.7628) (width 0.2) (layer F.Cu) (net 11))
   (segment (start 104.6988 108.7628) (end 107.0864 108.7628) (width 0.2) (layer F.Cu) (net 11))
-  (segment (start 114.646001 89.436501) (end 114.3635 89.154) (width 0.2) (layer F.Cu) (net 11))
-  (segment (start 114.3635 89.154) (end 112.9792 89.154) (width 0.2) (layer F.Cu) (net 11))
-  (segment (start 112.9792 89.154) (end 112.4712 89.662) (width 0.2) (layer F.Cu) (net 11))
+  (segment (start 114.646001 89.436501) (end 114.3508 89.1032) (width 0.2) (layer F.Cu) (net 11))
   (segment (start 116.2945 90.1865) (end 115.544501 89.436501) (width 0.2) (layer F.Cu) (net 11))
-  (segment (start 112.4712 89.662) (end 112.4712 92.9132) (width 0.2) (layer F.Cu) (net 11))
+  (segment (start 115.544501 89.436501) (end 114.646001 89.436501) (width 0.2) (layer F.Cu) (net 11))
   (segment (start 116.3495 103.051) (end 116.8745 103.051) (width 0.2) (layer F.Cu) (net 12))
   (segment (start 109.6015 103.051) (end 116.3495 103.051) (width 0.2) (layer F.Cu) (net 12))
@@
   (segment (start 100.043 105.918) (end 98.806 105.918) (width 0.6) (layer F.Cu) (net 50))
   (segment (start 98.806 105.918) (end 98.3615 106.3625) (width 0.6) (layer F.Cu) (net 50))
-  (segment (start 122.7745 103.051) (end 123.9234 103.051) (width 0.2) (layer F.Cu) (net 50))
   (segment (start 118.8245 99.776) (end 118.872 99.7285) (width 0.2) (layer F.Cu) (net 50))
   (segment (start 118.8245 100.301) (end 118.8245 99.776) (width 0.2) (layer F.Cu) (net 50))
@@
   (via (at 90.0176 92.9132) (size 0.6) (drill 0.3) (layers F.Cu B.Cu) (net 50))
   (via (at 92.5068 89.6112) (size 0.6) (drill 0.3) (layers F.Cu B.Cu) (net 50))
-  (via (at 79.1464 102.8192) (size 0.6) (drill 0.3) (layers F.Cu B.Cu) (net 50))
-  (via (at 77.8256 103.632) (size 0.6) (drill 0.3) (layers F.Cu B.Cu) (net 50))
-  (via (at 79.1464 101.9556) (size 0.6) (drill 0.3) (layers F.Cu B.Cu) (net 50))
-  (via (at 77.8256 100.9904) (size 0.6) (drill 0.3) (layers F.Cu B.Cu) (net 50))
-  (via (at 79.1464 100.1776) (size 0.6) (drill 0.3) (layers F.Cu B.Cu) (net 50))
-  (via (at 77.8256 102.7684) (size 0.6) (drill 0.3) (layers F.Cu B.Cu) (net 50))
-  (via (at 79.1464 101.0412) (size 0.6) (drill 0.3) (layers F.Cu B.Cu) (net 50))
-  (via (at 77.8256 101.854) (size 0.6) (drill 0.3) (layers F.Cu B.Cu) (net 50))
-  (via (at 77.8256 104.4956) (size 0.6) (drill 0.3) (layers F.Cu B.Cu) (net 50))
-  (via (at 79.1464 103.6828) (size 0.6) (drill 0.3) (layers F.Cu B.Cu) (net 50))
-  (via (at 79.1464 104.6988) (size 0.6) (drill 0.3) (layers F.Cu B.Cu) (net 50))
-  (via (at 77.8764 99.9744) (size 0.6) (drill 0.3) (layers F.Cu B.Cu) (net 50))
-  (via (at 77.7748 108.1532) (size 0.6) (drill 0.3) (layers F.Cu B.Cu) (net 50))
-  (via (at 77.8256 105.3592) (size 0.6) (drill 0.3) (layers F.Cu B.Cu) (net 50))
-  (via (at 77.7748 109.0168) (size 0.6) (drill 0.3) (layers F.Cu B.Cu) (net 50))
-  (via (at 79.0956 109.0676) (size 0.6) (drill 0.3) (layers F.Cu B.Cu) (net 50))
-  (via (at 79.0956 107.3404) (size 0.6) (drill 0.3) (layers F.Cu B.Cu) (net 50))
-  (via (at 79.0956 106.426) (size 0.6) (drill 0.3) (layers F.Cu B.Cu) (net 50))
-  (via (at 79.0956 108.204) (size 0.6) (drill 0.3) (layers F.Cu B.Cu) (net 50))
-  (via (at 77.7748 107.2388) (size 0.6) (drill 0.3) (layers F.Cu B.Cu) (net 50))
-  (via (at 77.7748 106.3752) (size 0.6) (drill 0.3) (layers F.Cu B.Cu) (net 50))
-  (via (at 79.0956 105.5624) (size 0.6) (drill 0.3) (layers F.Cu B.Cu) (net 50))
-  (via (at 77.7748 109.8804) (size 0.6) (drill 0.3) (layers F.Cu B.Cu) (net 50))
   (via (at 86.2965 114.427) (size 0.6) (drill 0.3) (layers F.Cu B.Cu) (net 50))
   (via (at 86.36 110.6932) (size 0.6) (drill 0.3) (layers F.Cu B.Cu) (net 50))
@@
   (via (at 95.1484 134.2644) (size 0.6) (drill 0.3) (layers F.Cu B.Cu) (net 50))
   (via (at 95.8596 133.6548) (size 0.6) (drill 0.3) (layers F.Cu B.Cu) (net 50))
+  (segment (start 122.7745 103.051) (end 123.9234 103.051) (width 0.2) (layer F.Cu) (net 50))
+  (segment (start 125.0161 104.6771) (end 125.5051 104.6771) (width 0.2) (layer F.Cu) (net 50))
+  (segment (start 124.6661 104.1146) (end 124.6661 104.3271) (width 0.2) (layer F.Cu) (net 50))
+  (segment (start 124.6661 104.3271) (end 125.0161 104.6771) (width 0.2) (layer F.Cu) (net 50))
+  (segment (start 125.5051 104.6771) (end 125.6284 104.8004) (width 0.2) (layer F.Cu) (net 50))
+  (segment (start 124.6632 102.6668) (end 124.3076 102.6668) (width 0.2) (layer F.Cu) (net 50))
+  (segment (start 123.9234 103.051) (end 124.5616 102.4128) (width 0.3) (layer F.Cu) (net 50))
   (zone (net 7) (net_name +3V3) (layer B.Cu) (hatch edge 0.508)
     (priority 1)

Commit message: Gerando GRBs
Parts:
- R13: moved to F.Cu
- moved C3 2.67 mm to (119.1, 97.0), turned to 180 degrees
- moved L2 0.78 mm to (117.9, 95.9), turned to 0 degrees
Routing:
- net Net-(C3-Pad2): track 6.94 -> 4.52 mm
- net +3V3: track 134.7 -> 135.5 mm, vias 25 -> 26
- net Net-(D1-Pad2): track 2.08 -> 2.77 mm, vias 0 -> 1
- net GND: vias 533 -> 541

Commit message: corrigindo.
Parts:
- removed Display1: OLED, Medidor:OLED
- U1: footprint Medidor:INA219 -> Medidor:INAright
- moved U1 1.09 mm to (101.9, 104.6)
Routing:
- net +3V3: track 135.5 -> 104.8 mm
- net SCL: track 46.1 -> 15.9 mm
- net SDA: track 27.4 -> 15.0 mm
- net GND: track 18.3 -> 16.6 mm
- net Net-(C5-Pad2): track 3.07 -> 4.04 mm
- net Net-(C5-Pad1): track 3.12 -> 4.03 mm
