File: Medidor.kicad_pcb (KiCad board)
At the start: 2 copper layers, 58.9 x 47.1 mm, 45 parts, among them J1 TC2030-CTX-TAG_CONECT, SW1 Rotary_Encoder_Switch, SW2 SW_DPST_x2, U1 INA219-INA, U3 2450AT18D0100, X1 32MHz

Commit message: more replacement
Parts:
- added U10: spacer, Medidor:spacer, F.Cu at (85.5, 90.4)
- added U4: Fiducial, Fiducial:Fiducial_0.75mm_Mask1.5mm, F.Cu at (128.6, 90.2)
- added U5: Fiducial, Fiducial:Fiducial_0.75mm_Mask1.5mm, F.Cu at (139.6, 130.1)
- added U6: Fiducial, Fiducial:Fiducial_0.75mm_Mask1.5mm, F.Cu at (87.4, 128.8)
- added U7: spacer, Medidor:spacer, F.Cu at (140.9, 90.1)
- added U8: spacer, Medidor:spacer, F.Cu at (140.6, 134.2)
- added U9: spacer, Medidor:spacer, F.Cu at (85.6, 133.9)
- C14, C15, D1, R10, R11, R12, R13, R14, R9: moved to F.Cu
- moved U3 29.9 mm to (85.4, 119.8), turned to 90 degrees
- moved L2 19.4 mm to (116.1, 118.3), turned to 270 degrees
- moved C3 18.8 mm to (114.9, 118.3), turned to 270 degrees
- moved L1 16.3 mm to (116.1, 115.7), turned to 270 degrees
- moved R7 16.2 mm to (99.3, 118.7)
- moved R6 16.0 mm to (101.1, 118.2)
- moved X1 16.0 mm to (108.0, 117.1), turned to 90 degrees
- moved R8 16.0 mm to (101.1, 119.3)
- moved C1 15.9 mm to (108.9, 117.1), turned to 90 degrees
- moved C7 15.9 mm to (118.8, 112.9), turned to 180 degrees
- moved C2 15.0 mm to (104.6, 115.1), turned to 90 degrees
- moved C10 14.3 mm to (118.5, 111.6), turned to 180 degrees
- moved SW2 13.7 mm to (92.2, 118.1)
- moved C9 11.2 mm to (109.8, 113.9), turned to 0 degrees
- moved Screw_Terminal 10.6 mm to (135.8, 108.5), turned to 270 degrees
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- renumbered UART to U2, dc-dc to dc1
Connections:
- MCU1 pad 15: /TX -> Net-(MCU1-Pad15)
- MCU1 pad 16: /RX -> Net-(MCU1-Pad16)
- MCU1 pad 3: Net-(MCU1-Pad3) -> /TX
- MCU1 pad 38: Net-(MCU1-Pad38) -> RC1
- MCU1 pad 39: Net-(MCU1-Pad39) -> RC2
- MCU1 pad 4: RC3 -> /RX
- MCU1 pad 42: SDA -> LEDMCU
- MCU1 pad 43: SCL -> RC3
- MCU1 pad 5: RC2 -> Net-(MCU1-Pad5)
- MCU1 pad 6: RC1 -> Net-(MCU1-Pad6)
- MCU1 pad 8: LEDMCU -> SDA
- MCU1 pad 9: Net-(MCU1-Pad9) -> SCL
Routing:
- net RC3: track 0.00 -> 2.64 mm
