File: Medidor.sch (KiCad schematic (older format))
At the start: 45 parts, among them J1 TC2030-CTX-TAG_CONECT, SW1 Rotary_Encoder_Switch, SW2 SW_DPST_x2, U1 INA219-INA, U2 Serial, U3 2450AT18D0100, X1 32MHz

Commit message: more replacement
Parts:
- added U10, U7, U8, U9: spacer, Medidor:spacer, symbol medidor:spacer
- added U4, U5, U6: Fiducial, Fiducial:Fiducial_0.75mm_Mask1.5mm, symbol medidor:Fiducial
Connections:
- net LEDMCU: now also MCU1.42 (P0.30/AIN6); no longer MCU1.8 (P0.06)
- net RC1: now also MCU1.38 (P0.26); no longer MCU1.6 (P0.04/AIN2)
- net RC2: now also MCU1.39 (P0.27); no longer MCU1.5 (P0.03/AIN1)
- net RC3: now also MCU1.43 (P0.31/AIN7); no longer MCU1.4 (P0.02/AIN0)
- net RX: now also MCU1.4 (P0.02/AIN0); no longer MCU1.16 (P0.13)
- net SCL: now also MCU1.9 (P0.07); no longer MCU1.43 (P0.31/AIN7)
- net SDA: now also MCU1.8 (P0.06); no longer MCU1.42 (P0.30/AIN6)
- net TX: now also MCU1.3 (P0.01/XL2); no longer MCU1.15 (P0.12)
Changed lines of the file:
@@
 Wire Wire Line
 	5400 2500 5400 3550
-Text GLabel 5750 3050 2    50   Input ~ 0
+Text GLabel 4250 4550 0    50   Input ~ 0
 SDA
 Wire Wire Line
@@
 Wire Wire Line
 	5700 3050 5750 3050
-Text GLabel 5750 2900 2    50   Input ~ 0
+Text GLabel 4250 4650 0    50   Input ~ 0
 SCL
 Wire Wire Line
@@
 Wire Wire Line
 	3800 1400 3800 1550
-Text GLabel 4250 4550 0    50   Input ~ 0
+Text GLabel 5750 3050 2    50   Input ~ 0
 LEDMCU
 Wire Wire Line
@@
 ALIMENTAÇÂO
 NoConn ~ 4750 3950
-NoConn ~ 4750 4050
 NoConn ~ 4750 4450
-NoConn ~ 4750 4650
 NoConn ~ 4750 4750
 NoConn ~ 4750 4850
@@
 Wire Wire Line
 	2000 5500 2000 5400
-Text GLabel 4200 4350 0    50   Input ~ 0
+Text GLabel 6100 3350 2    50   Input ~ 0
 RC1
-Wire Wire Line
-	4200 4150 4750 4150
-Text GLabel 4200 4250 0    50   Input ~ 0
+Text GLabel 6050 3200 2    50   Input ~ 0
 RC2
-Wire Wire Line
-	4200 4250 4750 4250
 Text GLabel 1000 5450 0    50   Input ~ 0
 RC1
@@
 NoConn ~ 5200 5350
 Wire Wire Line
-	5300 5550 5300 5350
-Wire Wire Line
 	4300 6600 4200 6600
 Wire Wire Line
@@
 Wire Wire Line
 	9800 2050 10000 2050
-NoConn ~ 6100 3550
-NoConn ~ 6000 3550
 Wire Wire Line
 	1900 4650 1900 4450
@@
 Text Label 4500 6600 0    50   ~ 0
 RX
-Text Label 5300 5550 0    50   ~ 0
+Text Label 4650 4050 0    50   ~ 0
 TX
-Wire Wire Line
-	5400 5350 5400 5550
-Text Label 5400 5550 0    50   ~ 0
+Text Label 4650 4150 0    50   ~ 0
 RX
 Text GLabel 2200 4450 2    50   Input ~ 0
 RC3
-Text GLabel 4200 4150 0    50   Input ~ 0
+Text GLabel 5750 2900 2    50   Input ~ 0
 RC3
-Wire Wire Line
-	4200 4350 4750 4350
 Wire Notes Line
 	7600 5100 11150 5100
@@
 Wire Notes Line
 	3000 2200 4500 2200
+$Comp
+L medidor:Fiducial U4
+U 1 1 5D438E8C
+P 9350 3200
+F 0 "U4" H 9584 3246 50  0000 L CNN
+F 1 "Fiducial" H 9584 3155 50  0000 L CNN
+F 2 "Fiducial:Fiducial_0.75mm_Mask1.5mm" H 9350 3250 50  0001 C CNN
+F 3 "" H 9350 3250 50  0001 C CNN
+	1    9350 3200
+	1    0    0    -1
+$EndComp
+$Comp
+L medidor:Fiducial U6
+U 1 1 5D43A2B9
+P 10300 3200
+F 0 "U6" H 10534 3246 50  0000 L CNN
+F 1 "Fiducial" H 10534 3155 50  0000 L CNN
+F 2 "Fiducial:Fiducial_0.75mm_Mask1.5mm" H 10300 3250 50  0001 C CNN
+F 3 "" H 10300 3250 50  0001 C CNN
+	1    10300 3200
+	1    0    0    -1
+$EndComp
+$Comp
+L medidor:Fiducial U5
+U 1 1 5D43A693
+P 9800 3600
+F 0 "U5" H 10034 3646 50  0000 L CNN
+F 1 "Fiducial" H 10034 3555 50  0000 L CNN
+F 2 "Fiducial:Fiducial_0.75mm_Mask1.5mm" H 9800 3650 50  0001 C CNN
+F 3 "" H 9800 3650 50  0001 C CNN
+	1    9800 3600
+	1    0    0    -1
+$EndComp
+$Comp
+L medidor:spacer U7
+U 1 1 5D43D50E
+P 9650 4100
+F 0 "U7" H 9819 4146 50  0000 L CNN
+F 1 "spacer" H 9819 4055 50  0000 L CNN
+F 2 "Medidor:spacer" H 9650 4100 50  0001 C CNN
+F 3 "" H 9650 4100 50  0001 C CNN
+	1    9650 4100
+	1    0    0    -1
+$EndComp
+$Comp
+L medidor:spacer U9
+U 1 1 5D43E3DB
+P 10350 4100
+F 0 "U9" H 10519 4146 50  0000 L CNN
+F 1 "spacer" H 10519 4055 50  0000 L CNN
+F 2 "Medidor:spacer" H 10350 4100 50  0001 C CNN
+F 3 "" H 10350 4100 50  0001 C CNN
+	1    10350 4100
+	1    0    0    -1
+$EndComp
+$Comp
+L medidor:spacer U8
+U 1 1 5D43E795
+P 10000 4500
+F 0 "U8" H 10169 4546 50  0000 L CNN
+F 1 "spacer" H 10169 4455 50  0000 L CNN
+F 2 "Medidor:spacer" H 10000 4500 50  0001 C CNN
+F 3 "" H 10000 4500 50  0001 C CNN
+	1    10000 4500
+	1    0    0    -1
+$EndComp
+$Comp
+L medidor:spacer U10
+U 1 1 5D44398C
+P 9400 4550
+F 0 "U10" H 9569 4596 50  0000 L CNN
+F 1 "spacer" H 9569 4505 50  0000 L CNN
+F 2 "Medidor:spacer" H 9400 4550 50  0001 C CNN
+F 3 "" H 9400 4550 50  0001 C CNN
+	1    9400 4550
+	1    0    0    -1
+$EndComp
+Wire Wire Line
+	4250 4650 4750 4650
+Wire Wire Line
+	6050 3200 6000 3200
+Wire Wire Line
+	6000 3200 6000 3550
+Wire Wire Line
+	6100 3550 6100 3350
+NoConn ~ 4750 4250
+NoConn ~ 4750 4350
+Wire Wire Line
+	4750 4050 4650 4050
+Wire Wire Line
+	4750 4150 4650 4150
+NoConn ~ 5400 5350
+NoConn ~ 5300 5350
 $EndSCHEMATC
